File: banglet/eaglecad/dc5032018banglet.sch (EAGLE design)
At the start: 38 parts, among them J1 S2B-EH(LF)(SN), Q3 DMG3415U-7, U2 AP2112(3.3V), U3 MCP73831T-2ACI/OT, U4 CP2104, X1 32.768, X4 20329

Commit message: Added new part for LED strip connection
- Added new part to banglet library
- Replaced vias for the LED strip with new part

Eaglecad refuses to name the vias after the nets in the schematic

Signed-off-by: nisha <nishakumarx@gmail.com>
Parts:
- removed A0, GND, VLED: WIREPAD2,54/0,9, wirepad:WIREPAD2,54/0,9
- added LEDCONN: WS2812B-LED-STRIPLEDCONN, banglet:WS2812B-LED-STRIPLEDCONN
Connections:
- removed net N$3: JP3.2, VLED.P
- new net VLED: JP3.2, LEDCONN.1
- net A0: no longer A0.P
- net GND: no longer GND.P
Changed lines of the file:
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@@
 <part name="GND14" library="supply1" library_urn="urn:adsk.eagle:library:371" deviceset="GND" device=""/>
 <part name="GND15" library="supply1" library_urn="urn:adsk.eagle:library:371" deviceset="GND" device=""/>
-<part name="A0" library="wirepad" library_urn="urn:adsk.eagle:library:412" deviceset="WIREPAD" device="2,54/0,9"/>
-<part name="VLED" library="wirepad" library_urn="urn:adsk.eagle:library:412" deviceset="WIREPAD" device="2,54/0,9"/>
-<part name="GND" library="wirepad" library_urn="urn:adsk.eagle:library:412" deviceset="WIREPAD" device="2,54/0,9"/>
 <part name="X4" library="microbuilder" deviceset="MICRO-USB-SMD-B-(10118193-0001LF)-ADASYM" device="" value="20329"/>
 <part name="U$11" library="microbuilder" deviceset="GND" device=""/>
@@
 <part name="FD2" library="SparkFun-Aesthetics" library_urn="urn:adsk.eagle:library:507" deviceset="FIDUCIAL" device="UFIDUCIAL" package3d_urn="urn:adsk.eagle:package:37111/1"/>
 <part name="J1" library="banglet" deviceset="S2B-EH(LF)(SN)" device=""/>
+<part name="LEDCONN" library="banglet" deviceset="WS2812B-LED-STRIP" device="LEDCONN"/>
 </parts>
 <sheets>
@@
 <instance part="GND14" gate="1" x="38.1" y="25.4" rot="R90"/>
 <instance part="GND15" gate="1" x="22.86" y="-45.72"/>
-<instance part="A0" gate="G$1" x="-38.1" y="-15.24"/>
-<instance part="VLED" gate="G$1" x="-40.64" y="-45.72"/>
-<instance part="GND" gate="G$1" x="-45.72" y="10.16"/>
 <instance part="X4" gate="G$1" x="104.14" y="68.58" rot="R270"/>
 <instance part="U$11" gate="G$1" x="99.06" y="55.88"/>
@@
 <instance part="FD2" gate="G$1" x="66.04" y="-60.96"/>
 <instance part="J1" gate="G$1" x="63.5" y="58.42"/>
+<instance part="LEDCONN" gate="G$1" x="167.64" y="-22.86"/>
 </instances>
 <busses>
@@
 <wire x1="-27.94" y1="10.16" x2="-27.94" y2="12.7" width="0.1524" layer="91"/>
 <junction x="-27.94" y="12.7"/>
-<pinref part="GND" gate="G$1" pin="P"/>
 <wire x1="-43.18" y1="10.16" x2="-27.94" y2="10.16" width="0.1524" layer="91"/>
 <junction x="-27.94" y="10.16"/>
@@
 <pinref part="C2" gate="G$1" pin="2"/>
 <wire x1="-33.02" y1="-33.02" x2="-33.02" y2="-30.48" width="0.1524" layer="91"/>
+</segment>
+<segment>
+<wire x1="175.26" y1="-25.4" x2="180.34" y2="-25.4" width="0.1524" layer="91"/>
 </segment>
 </net>
@@
 <wire x1="-22.86" y1="-15.24" x2="-35.56" y2="-15.24" width="0.1524" layer="91"/>
 <label x="-35.56" y="-15.24" size="1.778" layer="95"/>
-<pinref part="A0" gate="G$1" pin="P"/>
+</segment>
+<segment>
+<wire x1="175.26" y1="-22.86" x2="180.34" y2="-22.86" width="0.1524" layer="91"/>
 </segment>
 </net>
@@
 </segment>
 </net>
-<net name="N$3" class="0">
-<segment>
-<pinref part="VLED" gate="G$1" pin="P"/>
+<net name="VLED" class="0">
+<segment>
 <pinref part="JP3" gate="G$1" pin="2"/>
 <wire x1="-38.1" y1="-45.72" x2="-35.56" y2="-45.72" width="0.1524" layer="91"/>
 </segment>
-</net>
+<segment>
+<pinref part="LEDCONN" gate="G$1" pin="1"/>
+<wire x1="175.26" y1="-20.32" x2="180.34" y2="-20.32" width="0.1524" layer="91"/>
+</segment>
+</net>

Commit message: connect led header in schematic and board
Connections:
- net A0: now also LEDCONN.2
- net GND: now also LEDCONN.3
Changed lines of the file:
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@@
 <segment>
 <wire x1="175.26" y1="-25.4" x2="180.34" y2="-25.4" width="0.1524" layer="91"/>
+<pinref part="LEDCONN" gate="G$1" pin="3"/>
 </segment>
 </net>
@@
 <segment>
 <wire x1="175.26" y1="-22.86" x2="180.34" y2="-22.86" width="0.1524" layer="91"/>
-</segment>
-</net>
+<pinref part="LEDCONN" gate="G$1" pin="2"/>
+</segment>
+</net>
